File: Hardware/Sensor/chamber.kicad_pcb (KiCad board)
At the start: 2 copper layers, 100 x 100 mm, 102 parts, among them J1 USB_B_Micro, J32 RF_Shield_Two_Pieces, J33 RF_Shield_Two_Pieces, J34 Conn_Coaxial, J51 Conn_02x05_Counter_Clockwise, J52 Conn_01x04, Q31 BC859, Q32 Q_NMOS_GDS, Q51 2N7002, Q52 Q_NPN_BEC, SW31 SW_DPDT_x2, SW32 SW_DPDT_x2, U31 MC34063AD, U32 LMC662, U33 LM358, U51 Opamp_Dual_Generic, U52 MCP3425A0T-ECH, U53 MCP3425A0T-ECH, U54 STM8S003F3P

Commit message: add draft of pcb with high voltage supply and opamp power supply
Parts:
- removed BT31: 2 x 3V6, Battery:BatteryHolder_Keystone_2466_1xAAA
- removed C1, C31, C35, C54, C55, C57: 100n, Capacitor_SMD:C_0805_2012Metric_Pad1.15x1.40mm_HandSolder
- removed C2: 100u/6V3, Capacitor_Tantalum_SMD:CP_EIA-3528-21_Kemet-B
- removed C32: 3n3, Capacitor_SMD:C_0805_2012Metric_Pad1.15x1.40mm_HandSolder
- removed C39: 10n, Capacitor_SMD:C_0805_2012Metric_Pad1.15x1.40mm_HandSolder
- removed C41, C43: 10n/600V, Capacitor_THT:C_Disc_D8.0mm_W2.5mm_P5.00mm
- removed C56: 10u, Capacitor_Tantalum_SMD:CP_EIA-3528-21_Kemet-B
- removed D1, D31, D35: red, LED_SMD:LED_0805_2012Metric
- removed D32: D_Schottky, Diode_SMD:D_SOT-23_ANK
- removed D33: 1N4007, Diode_THT:D_DO-41_SOD81_P10.16mm_Horizontal
- removed D34: 1N4007, Diode_THT:D_DO-41_SOD81_P5.08mm_Vertical_AnodeUp
- removed D50, D51: 1n148, Diode_SMD:D_MiniMELF
- removed J1: USB_B_Micro, Connector_USB:USB_Micro-B_Molex_47346-0001
- removed J32: RF_Shield_Two_Pieces, IonizationChamber:IonizationChamberHVShield
- removed J33: RF_Shield_Two_Pieces, IonizationChamber:IonizationChamberShield
- removed L31: 680m, Inductor_THT:L_Radial_L8.0mm_W8.0mm_P5.00mm_Neosid_NE-CPB-07E
- removed Q31: BC859, Package_TO_SOT_SMD:SOT-23
- removed Q32: Q_NMOS_GDS, Package_TO_SOT_THT:TO-220-3_Horizontal_TabDown
- removed Q51: 2N7002, Package_TO_SOT_SMD:SOT-23
- removed Q52: Q_NPN_BEC, Package_TO_SOT_SMD:SOT-323_SC-70_Handsoldering
- removed R1, R43, R44: 520R, Resistor_SMD:R_0805_2012Metric_Pad1.15x1.40mm_HandSolder
- removed R31: R22/0.5W, Resistor_THT:R_Axial_DIN0207_L6.3mm_D2.5mm_P5.08mm_Vertical
- removed R32: 10k, Resistor_SMD:R_0805_2012Metric_Pad1.15x1.40mm_HandSolder
- removed R33, R36, R37: 10M, Resistor_THT:R_Axial_DIN0207_L6.3mm_D2.5mm_P10.16mm_Horizontal
- removed R34, R54, R55, R56, R57, R58: 1k, Resistor_SMD:R_0805_2012Metric_Pad1.15x1.40mm_HandSolder
- removed R35: 30k, Resistor_SMD:R_0805_2012Metric_Pad1.15x1.40mm_HandSolder
- removed RV51: R_POT_TRIM, Potentiometer_THT:Potentiometer_Bourns_3296W_Vertical
- removed SW32: SW_DPDT_x2, IonizationChamber:SwitchButtonGeneric
- removed TP30: TestPoint, TestPoint:TestPoint_Loop_D2.60mm_Drill0.9mm_Beaded
- removed TP57: TestPoint, TestPoint:TestPoint_THTPad_1.0x1.0mm_Drill0.5mm
- removed U31: MC34063AD, Package_SO:SOIC-8_3.9x4.9mm_P1.27mm
- removed U51: Opamp_Dual_Generic, Package_SO:SOIC-8_3.9x4.9mm_P1.27mm
- removed U52: MCP3425A0T-ECH, Package_TO_SOT_SMD:SOT-23-6_Handsoldering
- added BT1: 2 x 3V6, Battery:BatteryHolder_Keystone_2466_1xAAA, F.Cu at (109.7, 219.5)
- added BT2: 3V6, IonizationChamber:MR18650BatteryHolder, F.Cu at (129.0, 139.7)
- added BT3: 2 x 3V6, Battery:BatteryHolder_Keystone_2466_1xAAA, F.Cu at (80.3, 219.5)
- added BT4: 3V6, IonizationChamber:MR18650BatteryHolder, F.Cu at (177.8, 139.7)
- added BT5: 3V6, IonizationChamber:MR18650BatteryHolder, F.Cu at (160.0, 139.7)
- added BT6: 2 x 3V6, Battery:BatteryHolder_Keystone_2466_1xAAA, F.Cu at (69.8, 146.6)
- added BT9: 2 x 3V6, Battery:BatteryHolder_Keystone_2466_1xAAA, F.Cu at (1.02, 133.9)
- added TH1: Thermistor, Resistor_SMD:R_0805_2012Metric, F.Cu at (248.4, 84.3)
- BT32: value 2 x 3V6 -> 3V6; footprint Battery:BatteryHolder_Keystone_2466_1xAAA -> IonizationChamber:MR18650BatteryHolder; moved to F.Cu
- C4, C5: value 0R resistor -> 10n
- C52: value 100n -> 680n
- D2: value LED -> yellow
- D3: value LED -> green
- D4: value LED -> red
- R42: value 22k -> 120k
- R52: value 22k -> 0R
- R53: value R -> 27k
- moved C33 94.8 mm to (77.5, 21.4)
- moved C40 94.8 mm to (74.9, 46.0)
- moved C45 94.8 mm to (95.5, 59.2)
- moved L32 94.8 mm to (74.4, 28.2)
- moved R38 94.8 mm to (68.4, 46.7)
- moved R41 94.8 mm to (92.2, 49.5)
- moved SW31 94.8 mm to (64.3, 21.8)
- moved U32 94.8 mm to (70.9, 47.8)
- moved U33 94.8 mm to (93.0, 54.2)
- moved V31 94.8 mm to (63.5, 42.2)
- moved C34 94.8 mm to (67.2, 27.4)
- moved C4 94.8 mm to (83.1, 43.7)
- moved C42 94.8 mm to (74.0, 41.9)
- moved C44 94.8 mm to (86.9, 52.3)
- moved C46 94.8 mm to (65.8, 46.7)
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Connections:
- BT32 pad 1: GND -> Net-(BT32-Pad1)
- C50 pad 2: VCC_5V -> +5V
- C51 pad 1: VCC_5V -> +5V
- C53 pad 2: /DataAcquisition/VCC_PROG -> +5V
- J51 pad 5: /DataAcquisition/VCC_PROG -> +5V
- R59 pad 2: VCC_5V -> +5V
- R60 pad 2: VCC_5V -> +5V
- TP31 pad 1: Net-(D34-Pad1) -> +BATT
- U53 pad 5: VCC_5V -> +5V
- U54 pad 1: /DataAcquisition/INT0 -> (no net)
- U54 pad 5: /DataAcquisition/RST_PEAK -> (no net)
- U54 pad 9: /DataAcquisition/VCC_PROG -> +5V
- V31 pad 1: Net-(D34-Pad1) -> +BATT
Routing:
- net VCC_5V: track 144.6 -> 0.00 mm, vias 4 -> 0
- net +5V: track 0.00 -> 110.2 mm, vias 0 -> 4
- net Net-(C2-Pad1): track 62.5 -> 0.00 mm
- net GND: track 484.6 -> 440.8 mm, vias 54 -> 36
- net Net-(L31-Pad1): track 42.1 -> 0.00 mm, vias 2 -> 0
- net /DataAcquisition/INT0: track 37.0 -> 0.00 mm, vias 2 -> 0
- net Net-(C39-Pad1): track 33.0 -> 0.00 mm
- net Net-(D32-Pad1): track 21.1 -> 0.00 mm
- net Net-(C41-Pad1): track 17.7 -> 0.00 mm
- net Net-(D32-Pad2): track 18.1 -> 0.69 mm, vias 2 -> 0
- net Net-(D33-Pad2): track 16.1 -> 0.00 mm
- net Net-(C54-Pad2): track 15.8 -> 0.00 mm
- net /DataAcquisition/VCC_PROG: track 14.8 -> 0.00 mm
- net Net-(R57-Pad2): track 12.5 -> 0.00 mm
- net analog_output: track 67.6 -> 55.2 mm
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Other:
- board text removed: "400V DC chamber polarization"

Commit message: draft of sensor pcb
Parts:
- removed BT1, BT3, BT6, BT9: 2 x 3V6, Battery:BatteryHolder_Keystone_2466_1xAAA
- removed BT2, BT32, BT4, BT5: 3V6, IonizationChamber:MR18650BatteryHolder
- removed C3, C4, C5: 10n, Capacitor_SMD:C_0805_2012Metric_Pad1.15x1.40mm_HandSolder
- removed C33, C34: 100u/16V, Capacitor_SMD:CP_Elec_6.3x5.4
- removed C40, C42, C44, C45, C53: 100n, Capacitor_SMD:C_0805_2012Metric_Pad1.15x1.40mm_HandSolder
- removed C46: not mounted, Capacitor_SMD:C_0805_2012Metric_Pad1.15x1.40mm_HandSolder
- removed C47, C48: 0R resistor, Capacitor_SMD:C_0805_2012Metric_Pad1.15x1.40mm_HandSolder
- removed C52: 680n, Capacitor_SMD:C_0805_2012Metric_Pad1.15x1.40mm_HandSolder
- removed J34: Conn_Coaxial, Connector_Coaxial:SMA_Molex_73251-2200_Horizontal
- removed J51: Conn_02x05_Counter_Clockwise, Connector_PinSocket_2.54mm:PinSocket_2x05_P2.54mm_Horizontal
- removed J52: Conn_01x04, Connector_PinSocket_2.54mm:PinSocket_1x04_P2.54mm_Horizontal
- removed L32, L33: u68, Inductor_SMD:L_1812_4532Metric_Pad1.30x3.40mm_HandSolder
- removed the R2 at (269.5, 91.5)
- removed the R3 at (255.7, 94.0)
- removed R38: 2*50G, Resistor_SMD:R_0805_2012Metric_Pad1.15x1.40mm_HandSolder
- removed R39, R41: 10k, Resistor_SMD:R_0805_2012Metric_Pad1.15x1.40mm_HandSolder
- removed the R4 at (255.7, 91.5)
- removed R40, R42: 120k, Resistor_SMD:R_0805_2012Metric_Pad1.15x1.40mm_HandSolder
- removed SW31: SW_DPDT_x2, Button_Switch_THT:SW_E-Switch_EG1271_DPDT
- removed TP31: TestPoint, TestPoint:TestPoint_Loop_D2.60mm_Drill0.9mm_Beaded
- removed TP52, TP53, TP54, TP55, TP56: TestPoint, TestPoint:TestPoint_THTPad_1.0x1.0mm_Drill0.5mm
- removed U32: LMC662, Package_DIP:DIP-8_W7.62mm
- removed U33: LM358, Package_SO:SOIC-8_3.9x4.9mm_P1.27mm
- removed U54: STM8S003F3P, Package_SO:TSSOP-20_4.4x6.5mm_P0.65mm
- removed V31: Nuclear-Radiation_Detector, IonizationChamber:IonizationChamberSensor
- added C10: not mounted, Capacitor_SMD:C_0805_2012Metric, F.Cu at (76.0, 47.2)
- added C11: 10n, Capacitor_SMD:C_0805_2012Metric, F.Cu at (80.1, 66.2)
- added C12: 100n, Capacitor_SMD:C_0805_2012Metric, F.Cu at (74.3, 71.5)
- added C13: 100n, Capacitor_SMD:C_0805_2012Metric, F.Cu at (72.0, 53.7)
- added C14: 0R resistor, Capacitor_SMD:C_0805_2012Metric, F.Cu at (76.0, 50.2)
- added C6: 0R resistor, Capacitor_SMD:C_0805_2012Metric, F.Cu at (80.5, 47.2)
- added C7: 100n, Capacitor_SMD:C_0805_2012Metric, F.Cu at (80.1, 63.2)
- added C8: 100n, Capacitor_SMD:C_0805_2012Metric, F.Cu at (74.3, 68.5)
- added C9: 10n, Capacitor_SMD:C_0805_2012Metric, F.Cu at (69.2, 73.5)
- added H1: MountingHole_Pad, MountingHole:MountingHole_3.5mm_Pad, F.Cu at (62.5, 113.5)
- added H2: MountingHole_Pad, MountingHole:MountingHole_3.5mm_Pad, F.Cu at (134.5, 113.5)
- added H3: MountingHole_Pad, MountingHole:MountingHole_3.5mm_Pad, F.Cu at (134.5, 29.5)
- added H4: MountingHole_Pad, MountingHole:MountingHole_3.5mm_Pad, F.Cu at (62.5, 29.5)
- added J1: Conn_01x15_Female, Connector_PinSocket_2.54mm:PinSocket_1x15_P2.54mm_Vertical, F.Cu at (127.5, 92.0)
- added J2: Conn_01x15_Female, Connector_PinSocket_2.54mm:PinSocket_1x15_P2.54mm_Vertical, F.Cu at (127.5, 115.5)
- added J3: RF_Shield_One_Piece, IonizationChamber:RFShield, F.Cu at (88.0, 88.4)
- added J4: Conn_Coaxial, Connector_Coaxial:SMA_Molex_73251-2200_Horizontal, F.Cu at (63.5, 95.0)
- added J5: Conn_01x03_Male, Connector_PinSocket_2.54mm:PinSocket_1x03_P2.54mm_Vertical, B.Cu at (138.1, 44.2)
- added J6: Conn_01x03_Male, Connector_PinSocket_2.54mm:PinSocket_1x03_P2.54mm_Vertical, B.Cu at (62.8, 65.8)
- added R10: 10k, Resistor_SMD:R_0805_2012Metric, F.Cu at (73.6, 74.5)
- added R11: 2*50G, Resistor_SMD:R_0805_2012Metric, F.Cu at (78.7, 69.2)
- added R12: 120k, Resistor_SMD:R_0805_2012Metric, F.Cu at (72.0, 56.6)
- added R13: 120k, Resistor_SMD:R_0805_2012Metric, F.Cu at (76.4, 53.2)
- added R14: 10k, Resistor_SMD:R_0805_2012Metric, F.Cu at (78.7, 72.1)
- added TP6: TestPoint, TestPoint:TestPoint_Loop_D2.60mm_Drill0.9mm_Beaded, F.Cu at (69.5, 69.5)
- added U1: Nucleo32, IonizationChamber:Nucleo32, F.Cu at (136.5, 94.5)
- added U3: LMC662, Package_DIP:DIP-8_W7.62mm, F.Cu at (68.6, 57.3)
- added U4: LM358, Package_SO:SOIC-8_3.9x4.9mm_P1.27mm, F.Cu at (69.6, 48.9)
- added V1: Nuclear-Radiation_Detector, IonizationChamber:IonizationChamberSensor, F.Cu at (89.5, 37.0)
- C2: renamed from C50; footprint Capacitor_SMD:C_0805_2012Metric_Pad1.15x1.40mm_HandSolder -> Capacitor_SMD:C_0805_2012Metric
- D3: value green -> red
- R1: renamed from R52; footprint Resistor_SMD:R_0805_2012Metric_Pad1.15x1.40mm_HandSolder -> Resistor_SMD:R_0805_2012Metric
- R2: renamed from R51; footprint Resistor_SMD:R_0805_2012Metric_Pad1.15x1.40mm_HandSolder -> Resistor_SMD:R_0805_2012Metric
- R3: renamed from R50; footprint Resistor_SMD:R_0805_2012Metric_Pad1.15x1.40mm_HandSolder -> Resistor_SMD:R_0805_2012Metric
- R4: renamed from R53; footprint Resistor_SMD:R_0805_2012Metric_Pad1.15x1.40mm_HandSolder -> Resistor_SMD:R_0805_2012Metric
- R7: renamed from R59; footprint Resistor_SMD:R_0805_2012Metric_Pad1.15x1.40mm_HandSolder -> Resistor_SMD:R_0805_2012Metric
- moved C1 199.6 mm to (76.4, 105.7)
- moved C2 199.6 mm to (76.4, 102.5)
- moved R1 199.6 mm to (80.8, 94.2)
- moved R2 199.6 mm to (79.8, 97.3)
- moved R3 199.6 mm to (79.8, 100.3)
- moved R4 199.6 mm to (78.3, 94.2)
- moved R7 199.6 mm to (70.0, 106.7)
- moved R8 199.6 mm to (70.9, 104.1)
- moved U2 199.6 mm to (75.8, 98.8)
- moved D1 189.3 mm to (81.3, 116.4), turned to 270 degrees
- moved D2 180.4 mm to (72.9, 116.4), turned to 270 degrees
- moved D3 171.1 mm to (81.2, 109.7), turned to 270 degrees
- moved TH1 166.5 mm to (83.1, 104.5)
- renumbered C51 to C1, D2 to D1, D4 to D2, R60 to R8, U53 to U2
Connections:
- D1 pad 2: Net-(D2-Pad2) -> (no net)
- D2 pad 2: Net-(D4-Pad2) -> (no net)
- D3 pad 2: Net-(D3-Pad2) -> (no net)
- TH1 pad 1: Net-(TH1-Pad1) -> (no net)
Routing:
- net GND: track 440.8 -> 0.00 mm, vias 36 -> 0
- net +5V: track 110.2 -> 0.00 mm, vias 4 -> 0
- net +BATT: track 74.9 -> 0.00 mm, vias 4 -> 0
- net analog_output: track 55.2 -> 0.00 mm, vias 2 -> 0
- net /DataAcquisition/SCL: track 46.5 -> 0.00 mm, vias 3 -> 0
- net -BATT: track 44.8 -> 0.00 mm, vias 2 -> 0
- net /DataAcquisition/SDA: track 36.4 -> 0.00 mm, vias 3 -> 0
- net Net-(BT32-Pad2): track 30.0 -> 0.00 mm
- net /DataAcquisition/SWIM: track 23.7 -> 0.00 mm
- net Net-(C46-Pad1): track 17.4 -> 0.00 mm
- net /DataAcquisition/RST: track 16.8 -> 0.00 mm
- net Net-(C34-Pad2): track 14.7 -> 0.00 mm, vias 1 -> 0
- net Net-(BT2-Pad1): track 13.6 -> 0.00 mm
- net /DataAcquisition/RX: track 12.7 -> 0.00 mm, vias 1 -> 0
- net Net-(C5-Pad2): track 12.5 -> 0.00 mm
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Other:
- board size 100 x 100 mm -> 83 x 95 mm
- board text added: "HV supply is to low"
- board text added: "Ionization Chamber Sensor rev5.0"
- board text added: "data acquisition"
- board text added: "opamp supply to low"
- board text removed: "ADC converter"
- board text removed: "HV power on/off"
- board text removed: "HV+ADC power"
- board text removed: "Ionization Chamber Sensor rev4.0"
- board text removed: "power on"

Commit message: draft of routing of sensor
Parts:
- added BZ1: Buzzer, IonizationChamber:LPT1440S-HS-05-4.0-12-R, B.Cu at (79.9, 111.1)
- added C3: 100n, Capacitor_SMD:C_0805_2012Metric, F.Cu at (65.4, 65.2)
- added C4: 100n, Capacitor_SMD:C_0805_2012Metric, F.Cu at (65.4, 61.3)
- added C5: CP, Capacitor_SMD:CP_Elec_6.3x5.8, F.Cu at (72.5, 66.9)
- added J7: Conn_01x04_Female, Connector_PinSocket_2.54mm:PinSocket_1x04_P2.54mm_Vertical, F.Cu at (61.1, 101.2)
- added Q1: Q_PMOS_GDS, Package_TO_SOT_SMD:SOT-23, F.Cu at (62.8, 72.5)
- added Q2: Q_PMOS_GDS, Package_TO_SOT_SMD:SOT-23, F.Cu at (137.8, 49.9)
- added Q3: Q_NMOS_GDS, Package_TO_SOT_SMD:SOT-23, F.Cu at (67.7, 72.5)
- added Q4: Q_NMOS_GDS, Package_TO_SOT_SMD:SOT-23, F.Cu at (137.8, 55.0)
- added R15: TBD, Resistor_SMD:R_0805_2012Metric, F.Cu at (136.0, 52.6)
- added R16: TBD, Resistor_SMD:R_0805_2012Metric, F.Cu at (67.4, 75.3)
- added R17: TBD, Resistor_SMD:R_0805_2012Metric, F.Cu at (136.7, 58.0)
- added R5: TBD, Resistor_SMD:R_0805_2012Metric, F.Cu at (65.0, 69.5)
- added R6: TBD, Resistor_SMD:R_0805_2012Metric, F.Cu at (137.7, 47.1)
- added R9: TBD, Resistor_SMD:R_0805_2012Metric, F.Cu at (63.2, 75.3)
- C10: value not mounted -> CP; footprint Capacitor_SMD:C_0805_2012Metric -> Capacitor_SMD:CP_Elec_6.3x5.8
- D1: value yellow -> red
- H1, H2, H3, H4: value MountingHole_Pad -> MountingHole; footprint MountingHole:MountingHole_3.5mm_Pad -> MountingHole:MountingHole_3.5mm
- moved H4 110.6 mm to (134.4, 113.5)
- moved H3 110.6 mm to (62.5, 113.5)
- moved H2 84.1 mm to (135.4, 29.4)
- moved H1 84.0 mm to (64.2, 29.5)
- moved TP6 69.3 mm to (129.9, 35.4)
- moved C12 31.1 mm to (82.7, 41.5), turned to 180 degrees
- moved U4 30.7 mm to (81.1, 77.3)
- moved C13 28.3 mm to (79.6, 80.9)
- moved R14 28.0 mm to (71.5, 45.1)
- moved C9 25.4 mm to (70.5, 48.1), turned to 270 degrees
- moved C6 24.6 mm to (79.2, 71.8), turned to 180 degrees
- moved R11 19.6 mm to (85.2, 50.7), turned to 90 degrees
- moved R12 19.6 mm to (76.0, 75.8), turned to 270 degrees
- moved U3 15.1 mm to (82.7, 51.7), turned to 180 degrees
- moved C10 12.8 mm to (70.0, 58.5), turned to 90 degrees
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Connections:
- net Net-(J1-Pad10) renamed BATTERY_MEASSURE_ENA
- net Net-(J1-Pad11) renamed BATTERY_MEASSURE_VALUE
- net Net-(J1-Pad12) renamed CHAMBER_VOLTAGE_MEASSURE_VALUE
- net Net-(J1-Pad13) renamed CHAMBER_VOLTAGE_MEASSURE_ENA
- C10 pad 1: Net-(C10-Pad1) -> GND
- C10 pad 2: Net-(C10-Pad2) -> +BATT
- H1 pad 1: GND -> (no net)
- H2 pad 1: GND -> (no net)
- H3 pad 1: GND -> (no net)
- H4 pad 1: GND -> (no net)
- J5 pad 1: (no net) -> /AnalogFrontend/CHAMBER_VOLTAGE
- J6 pad 1: (no net) -> -BATT
- J6 pad 2: (no net) -> GND
- J6 pad 3: (no net) -> +BATT
- R11 pad 1: Net-(C10-Pad1) -> Net-(R11-Pad1)
- R11 pad 2: Net-(C10-Pad2) -> Net-(R11-Pad2)
- TP6 pad 1: +BATT -> /AnalogFrontend/CHAMBER_VOLTAGE
- U3 pad 1: Net-(C10-Pad1) -> Net-(R11-Pad1)
- U3 pad 2: Net-(C10-Pad2) -> Net-(R11-Pad2)
- U3 pad 5: Net-(C10-Pad1) -> Net-(R11-Pad1)
- V1 pad 1: +BATT -> /AnalogFrontend/CHAMBER_VOLTAGE
- V1 pad 2: Net-(C10-Pad2) -> Net-(R11-Pad2)
Routing:
- net GND: track 0.00 -> 116.0 mm
- net CHAMBER_VOLTAGE_MEASSURE_ENA: track 0.00 -> 74.5 mm
- net -BATT: track 0.00 -> 50.9 mm
- net /AnalogFrontend/CHAMBER_VOLTAGE: track 0.00 -> 24.3 mm
- net +BATT: track 0.00 -> 19.8 mm
- net Net-(R11-Pad1): track 0.00 -> 16.3 mm, vias 0 -> 2
- net Net-(C11-Pad1): track 0.00 -> 8.87 mm
- net Net-(Q2-Pad1): track 0.00 -> 7.00 mm
- net Net-(C9-Pad1): track 0.00 -> 6.98 mm
- net Net-(Q1-Pad1): track 0.00 -> 6.06 mm
- net CHAMBER_VOLTAGE_MEASSURE_VALUE: track 0.00 -> 5.18 mm
- net Net-(C11-Pad2): track 0.00 -> 4.82 mm
- net Net-(C6-Pad1): track 0.00 -> 4.63 mm
- net Net-(Q1-Pad3): track 0.00 -> 2.98 mm
- net Net-(R11-Pad2): track 0.00 -> 2.79 mm
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